File: Sensor_Current.sch (KiCad schematic (older format))
At the start: 71 parts, among them IC1 ATmega328, J1 Conn_DUT_A, J10 Conn_DUT_F, J11 Conn_DUT_G, J12 Conn_DUT_H, J13 Conn_SD_Breakout, J2 Conn_DUT_B, J3 Conn_DUT_C, J4 Conn_DUT_C, J5 Conn_FTDI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

Commit message: Updated PCB layout
Parts:
- removed C10, C11, C2, C3, C4, C8, C9: C, symbol CE_Capacitor:C
- BT1: footprint (none) -> Battery:BatteryHolder_Keystone_3034_1x20mm
- C1, C5, C6, C7: footprint (none) -> Capacitor_SMD:C_1206_3216Metric_Pad1.42x1.75mm_HandSolder
- D1: footprint (none) -> LED_SMD:LED_1206_3216Metric_Pad1.42x1.75mm_HandSolder
- J8: footprint Connector_PinHeader_2.54mm:PinHeader_1x10_P2.54mm_Vertical -> Connector_PinSocket_2.54mm:PinSocket_2x05_P2.54mm_Vertical
- RV1: footprint (none) -> Potentiometer_THT:Potentiometer_Bourns_3386F_Vertical
- SW1: footprint (none) -> Connector_PinHeader_2.54mm:PinHeader_1x02_P2.54mm_Vertical
- SW2, SW3: footprint (none) -> Button_Switch_SMD:SW_SPDT_PCM12
- TP_DB0, TP_DB1, TP_DB2, TP_DB3: footprint (none) -> TestPoint:TestPoint_Pad_D1.0mm
- Y1: footprint (none) -> Crystal:Crystal_HC49-U_Vertical
Other:
- note added: "Microcontroller"
- note added: "Power Management"
- note removed: "Power"
- moved on the sheet: BT1, C1, C5, C6, C7, D1, H1, H2, H3, H4, IC1, J13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
